Commit message: Change slightly the base position.

File: teststand_description/urdf/teststand.urdf.xacro (robot description, xacro)
@@ -21,5 +21,5 @@
   <link name="base_link">
     <inertial>
-        <origin rpy="0 0 0" xyz="0 0 ${base_h/2.}"/>
+        <origin rpy="0 0 0" xyz="0 0 0"/>
         <mass value="${base_m}"/>
         <inertia ixx="${1./12. * base_m * (base_h*base_h + base_w*base_w)}"
@@ -30,5 +30,5 @@
     </inertial>
     <visual>
-        <origin rpy="0 0 0" xyz="0 0 ${base_h/2.}"/>
+        <origin rpy="0 0 0" xyz="0 ${-base_w/2.} ${base_h/3.}"/>
         <geometry>
           <mesh filename="package://teststand_description/meshes/cube.obj" scale="${base_l} ${base_w} ${base_h}"/>
@@ -39,5 +39,5 @@
     </visual>
     <collision>
-        <origin rpy="0 0 0" xyz="0 0 ${base_h/2.}"/>
+        <origin rpy="0 0 0" xyz="0 ${-base_w/2.} ${base_h/3.}"/>
         <geometry>
             <box size="${base_l} ${base_w} ${base_h}"/>
