Commit message: Update URDF files (working both with simulation and hardware)
Signed-off-by: Victor T. N <victortn21@hotmail.com>

File: teststand_description/urdf/leg.xacro (robot description, xacro)
@@ -66,5 +66,5 @@
       </contact>
     </link> <!-- END UPPER LEG LINK -->
-    <!-- KFE: Joint between the upper leg and the lower leg -->
+    <!-- KFE Joint between the upper leg and the lower leg -->
     <joint name="${prefix}KFE" type="revolute">
       <parent link="${prefix}upperleg"/>
@@ -114,5 +114,5 @@
       </contact>
     </link> <!-- END LOWER LEG LINK -->
-    <!-- KFE: Joint between the upper leg and the lower leg -->
+    <!-- KFE Joint between the upper leg and the lower leg -->
     <joint name="${prefix}END" type="fixed">
       <parent link="${prefix}shank"/>

File: teststand_description/urdf/ros2_control.xacro (robot description, xacro)
@@ -1,34 +1,90 @@
 <?xml version="1.0"?>
 <robot xmlns:xacro="http://www.ros.org/wiki/xacro">
-    <ros2_control name="GazeboSimSystem" type="system">
-        <hardware>
-            <plugin>gz_ros2_control/GazeboSimSystem</plugin>
-        </hardware>
-        <joint name="joint_z">
-            <command_interface name="position"/>
+    <xacro:if value="${simulation}">
+        <xacro:property name="ros2_control_system" value="GazeboSimSystem"/>
+    </xacro:if>
+    <xacro:unless value="${simulation}">
+        <xacro:property name="ros2_control_system" value="SystemOdriHardware"/>
+    </xacro:unless>
+    <ros2_control name="${ros2_control_system}" type="system">
+        <xacro:if value="${simulation}">
+            <hardware>
+                <plugin>gz_ros2_control/GazeboSimSystem</plugin>
+            </hardware>
+        </xacro:if>
+        <xacro:unless value="${simulation}">
+            <hardware>
+                <plugin>ros2_control_odri/SystemOdriHardware</plugin>
+                <xacro:property name="teststand_config_yaml" value="$(find teststand_hw)/config/teststand_config.yaml"/>
+                <param name="odri_config_yaml">${teststand_config_yaml}</param>
+                <param name="desired_starting_position">0.0 0.0</param>
+                <param name="default_joint_cmd">HFE 0.0 0.0 0.0 3.0 0.05 KFE 0.0 0.0 0.0 3.0 0.05</param>
+                <param name="default_joint_state">HFE 0.0 0.0 0.0 3.0 0.05 KFE 0.0 0.0 0.0 3.0 0.05</param>
+            </hardware>
+        </xacro:unless>
+        <joint name="HFE">
+            <command_interface name="position">
+                <param name="min">-0.9</param>
+                <param name="max">0.9</param>
+            </command_interface>
+            <command_interface name="velocity">
+                <param name="min">-1</param>
+                <param name="max">1</param>
+            </command_interface>
+            <command_interface name="effort">
+                <param name="min">-1</param>
+                <param name="max">1</param>
+            </command_interface>
+            <command_interface name="gain_kp">
+                <param name="min">-1000</param>
+                <param name="max">1000</param>
+            </command_interface>
+            <command_interface name="gain_kd">
+                <param name="min">-1000</param>
+                <param name="max">1000</param>
+            </command_interface>
             <state_interface name="position"/>
             <state_interface name="velocity"/>
             <state_interface name="effort"/>
+            <state_interface name="gain_kp"/>
+            <state_interface name="gain_kd"/>
         </joint>
-        <joint name="HFE">
-            <command_interface name="position"/>
+        <joint name="KFE">
+            <command_interface name="position">
+                <param name="min">-0.9</param>
+                <param name="max">0.9</param>
+            </command_interface>
+            <command_interface name="velocity">
+                <param name="min">-1</param>
+                <param name="max">1</param>
+            </command_interface>
+            <command_interface name="effort">
+                <param name="min">-1</param>
+                <param name="max">1</param>
+            </command_interface>
+            <command_interface name="gain_kp">
+                <param name="min">-1000</param>
+                <param name="max">1000</param>
+            </command_interface>
+            <command_interface name="gain_kd">
+                <param name="min">-1000</param>
+                <param name="max">1000</param>
+            </command_interface>
             <state_interface name="position"/>
             <state_interface name="velocity"/>
             <state_interface name="effort"/>
-        </joint>
-        <joint name="KFE">
-            <command_interface name="position"/>
-            <state_interface name="position"/>
-            <state_interface name="velocity"/>
-            <state_interface name="effort"/>
+            <state_interface name="gain_kp"/>
+            <state_interface name="gain_kd"/>
         </joint>
     </ros2_control>
-    <gazebo>
-        <plugin filename="libgz_ros2_control-system" name="gz_ros2_control::GazeboSimROS2ControlPlugin">
-            <robot_param>robot_description</robot_param>
-            <robot_param_node>robot_state_publisher</robot_param_node>
-            <parameters>$(find teststand_control)/config/controllers.yaml</parameters>
-            <controller_manager_prefix_node_name>controller_manager</controller_manager_prefix_node_name>
-        </plugin>
-    </gazebo>
+    <xacro:if value="${simulation}">
+        <gazebo>
+            <plugin filename="libgz_ros2_control-system" name="gz_ros2_control::GazeboSimROS2ControlPlugin">
+                <robot_param>robot_description</robot_param>
+                <robot_param_node>robot_state_publisher</robot_param_node>
+                <parameters>$(find teststand_control)/config/controllers.yaml</parameters>
+                <controller_manager_prefix_node_name>controller_manager</controller_manager_prefix_node_name>
+            </plugin>
+        </gazebo>
+    </xacro:if>
 </robot>

File: teststand_description/urdf/teststand.urdf.xacro (robot description, xacro)
@@ -1,8 +1,7 @@
 <?xml version="1.0" ?>
-<robot name="teststand"
-  xmlns:controller="http://playerstage.sourceforge.net/gazebo/xmlschema/#controller"
-  xmlns:interface="http://playerstage.sourceforge.net/gazebo/xmlschema/#interface"
-  xmlns:sensor="http://playerstage.sourceforge.net/gazebo/xmlschema/#sensor"
-  xmlns:xacro="http://playerstage.sourceforge.net/gazebo/xmlschema/#interface">
+<robot name="teststand" xmlns:xacro="http://www.ros.org/wiki/xacro">
+  <!-- This argument controls which hardware interface plugins are loaded -->
+  <xacro:arg name="simulation" default="false"/>
+  <xacro:property name="simulation" value="$(arg simulation)"/>
   <xacro:property name="base_w" value=".1" />
   <xacro:property name="base_l" value=".2" />
